Commit message: add gazebo config

File: demobot2_description/urdf/circularbot/circularbot_essential.xacro (robot description, xacro)
@@ -131,12 +131,3 @@
     </joint>
   </xacro:macro>
-    <!-- Transmission is important to link the joints and the controller -->
-    <!-- <transmission name="${lr}_wheel_joint_trans">
-      <type>transmission_interface/SimpleTransmission</type>
-      <joint name="${lr}_wheel_joint" />
-      <actuator name="${lr}_wheel_joint_motor">
-        <hardwareInterface>EffortJointInterface</hardwareInterface>
-        <mechanicalReduction>1</mechanicalReduction>
-      </actuator>
-    </transmission> -->
 </robot>

File: demobot2_description/urdf/cubicbot/cubicbot_essential.xacro (robot description, xacro)
@@ -132,12 +132,3 @@
     </joint>
   </xacro:macro>
-    <!-- Transmission is important to link the joints and the controller -->
-    <!-- <transmission name="${lr}_wheel_joint_trans">
-      <type>transmission_interface/SimpleTransmission</type>
-      <joint name="${lr}_wheel_joint" />
-      <actuator name="${lr}_wheel_joint_motor">
-        <hardwareInterface>EffortJointInterface</hardwareInterface>
-        <mechanicalReduction>1</mechanicalReduction>
-      </actuator>
-    </transmission> -->
 </robot>

File: demobot2_description/urdf/demobot/demobot_essential.xacro (robot description, xacro)
@@ -86,13 +86,4 @@
       <dynamics damping="0.0" friction="0.1"/>
     </joint>
-    <!-- Transmission is important to link the joints and the controller -->
-    <!-- <transmission name="${lr}_wheel_joint_trans">
-      <type>transmission_interface/SimpleTransmission</type>
-      <joint name="${lr}_wheel_joint" />
-      <actuator name="${lr}_wheel_joint_motor">
-        <hardwareInterface>EffortJointInterface</hardwareInterface>
-        <mechanicalReduction>1</mechanicalReduction>
-      </actuator>
-    </transmission> -->
   </xacro:macro>
 </robot>

File: demobot2_description/urdf/demobot/demobot_urdf.xacro (robot description, xacro)
@@ -1,4 +1,4 @@
 <?xml version="1.0"?>
-<robot name="demobot" xmlns:xacro="http://www.ros.org/wiki/xacro">
+<robot name="demobot_urdf" xmlns:xacro="http://www.ros.org/wiki/xacro">
   <xacro:include filename="$(find demobot2_description)/urdf/demobot/demobot_essential.xacro" />
   <link name="base_footprint"/>

Commit message: update urdf file

File: demobot2_description/urdf/circularbot/circularbot_essential.xacro (robot description, xacro)
@@ -103,4 +103,33 @@
     </joint>
   </xacro:macro>
+  <!-- Visualization for real robot -->
+  <xacro:macro name="fixed_wheel" params="lr parent dir z_offset roll"> <!-- lr: left, right -->
+    <link name="${lr}_wheel_link">
+      <visual>
+        <origin xyz="0 0 0" rpy="0 0 0 " />
+        <geometry>
+          <cylinder length="${wheel_height}" radius="${wheel_radius}" />
+        </geometry>
+        <material name="Black" />
+      </visual>
+      <collision>
+        <origin xyz="0 0 0" rpy="0 0 0 " />
+        <geometry>
+          <cylinder length="${wheel_height}" radius="${wheel_radius}" />
+        </geometry>
+      </collision>
+      <inertial>
+        <mass value="${wheel_mass}" />
+        <origin xyz="0 0 0" />
+        <xacro:cylinder_inertia  m="${wheel_mass}" r="${wheel_radius}" h="${wheel_height}" />
+      </inertial>
+    </link>
+    <joint name="${lr}_wheel_joint" type="fixed">
+      <parent link="${parent}"/>
+      <child link="${lr}_wheel_link"/>
+      <origin xyz="0 ${dir * wheel_spacing / 2} ${z_offset}" rpy="${roll} 0 0" />
+      <axis xyz="0 0 1" rpy="0 0 0" />
+    </joint>
+  </xacro:macro>
   <xacro:macro name="caster" params="fb parent dir z_offset roll color"> <!-- fb: front, back -->
     <link name="${fb}_caster_link">

File: demobot2_description/urdf/circularbot/circularbot_gazebo.urdf (robot description, URDF)
Before this commit: robot circularbot_gazebo, 10 links, 9 joints
Joints:
- joint lidar_joint: origin xyz=0 0 0.5 rpy=0 0 0 -> xyz=0 0 -0.32 rpy=0 0 0

File: demobot2_description/urdf/circularbot/circularbot_gazebo.xacro (robot description, xacro)
@@ -124,8 +124,8 @@
       <publish_odom>true</publish_odom>
       <publish_odom_tf>true</publish_odom_tf>
-      <publish_wheel_tf>false</publish_wheel_tf>
+      <publish_wheel_tf>true</publish_wheel_tf>
       <odometry_topic>odom</odometry_topic>
       <odometry_frame>odom</odometry_frame>
-      <robot_base_frame>base_footprint</robot_base_frame> <!-- will pub tf between /odom and /base_footprint-->
+      <robot_base_frame>base_footprint</robot_base_frame>
     </plugin>
   </gazebo>

File: demobot2_description/urdf/circularbot/circularbot_urdf_fixed.urdf (robot description, URDF)
Before this commit: robot circularbot_urdf, 10 links, 9 joints
Joints:
- joint left_wheel_joint: limit effort=100 velocity=100 -> (none); type continuous -> fixed
- joint lidar_joint: origin xyz=0 0 0.5 rpy=0 0 0 -> xyz=0 0 -0.32 rpy=0 0 0
- joint right_wheel_joint: limit effort=100 velocity=100 -> (none); type continuous -> fixed

File: demobot2_description/urdf/circularbot/circularbot_urdf_fixed.xacro (robot description, xacro)
@@ -109,6 +109,6 @@
   </joint>
   <!-- Wheels -->
-  <xacro:wheel lr="left" parent="base_link" dir="1" z_offset="-0.43" roll="${-1.0 * M_PI_2}"/>
-  <xacro:wheel lr="right" parent="base_link" dir="-1" z_offset="-0.43" roll="${-1.0 * M_PI_2}"/>
+  <xacro:fixed_wheel lr="left" parent="base_link" dir="1" z_offset="-0.43" roll="${-1.0 * M_PI_2}"/>
+  <xacro:fixed_wheel lr="right" parent="base_link" dir="-1" z_offset="-0.43" roll="${-1.0 * M_PI_2}"/>
   <!-- Casters -->
   <xacro:caster fb="front" parent="base_link" dir="1" z_offset="-0.449" roll="0" color="Red"/>

File: demobot2_description/urdf/cubicbot/cubicbot_essential.xacro (robot description, xacro)
@@ -104,4 +104,33 @@
     </joint>
   </xacro:macro>
+  <!-- Visualization for real robot -->
+  <xacro:macro name="fixed_wheel" params="lr parent dir z_offset roll"> <!-- lr: left, right -->
+    <link name="${lr}_wheel_link">
+      <visual>
+        <origin xyz="0 0 0" rpy="0 0 0 " />
+        <geometry>
+          <cylinder length="${wheel_height}" radius="${wheel_radius}" />
+        </geometry>
+        <material name="Black" />
+      </visual>
+      <collision>
+        <origin xyz="0 0 0" rpy="0 0 0 " />
+        <geometry>
+          <cylinder length="${wheel_height}" radius="${wheel_radius}" />
+        </geometry>
+      </collision>
+      <inertial>
+        <mass value="${wheel_mass}" />
+        <origin xyz="0 0 0" />
+        <xacro:cylinder_inertia  m="${wheel_mass}" r="${wheel_radius}" h="${wheel_height}" />
+      </inertial>
+    </link>
+    <joint name="${lr}_wheel_joint" type="fixed">
+      <parent link="${parent}"/>
+      <child link="${lr}_wheel_link"/>
+      <origin xyz="0 ${dir * wheel_spacing / 2} ${z_offset}" rpy="${roll} 0 0" />
+      <axis xyz="0 0 1" rpy="0 0 0" />
+    </joint>
+  </xacro:macro>
   <xacro:macro name="caster" params="fb parent dir z_offset roll color"> <!-- fb: front, back -->
     <link name="${fb}_caster_link">

File: demobot2_description/urdf/cubicbot/cubicbot_gazebo.urdf (robot description, URDF)
Before this commit: robot cubicbot_gazebo, 10 links, 9 joints
Joints:
- joint lidar_joint: origin xyz=0 0 0.5 rpy=0 0 0 -> xyz=0 0 -0.32 rpy=0 0 0

File: demobot2_description/urdf/cubicbot/cubicbot_gazebo.xacro (robot description, xacro)
@@ -124,8 +124,8 @@
       <publish_odom>true</publish_odom>
       <publish_odom_tf>true</publish_odom_tf>
-      <publish_wheel_tf>false</publish_wheel_tf>
+      <publish_wheel_tf>true</publish_wheel_tf>
       <odometry_topic>odom</odometry_topic>
       <odometry_frame>odom</odometry_frame>
-      <robot_base_frame>base_footprint</robot_base_frame> <!-- will pub tf between /odom and /base_footprint-->
+      <robot_base_frame>base_footprint</robot_base_frame>
     </plugin>
   </gazebo>

File: demobot2_description/urdf/cubicbot/cubicbot_urdf.xacro (robot description, xacro)
@@ -96,5 +96,5 @@
     <parent link="base_link"/>
     <child link="lidar_link"/>
-    <origin xyz="0 0 0.5" rpy="0 0 0"/> <!-- default z: -0.32 -->
+    <origin xyz="0 0 -0.32" rpy="0 0 0"/> <!-- default z: -0.32 -->
   </joint>
   <joint name="camera_joint" type="fixed">

File: demobot2_description/urdf/cubicbot/cubicbot_urdf_fixed.urdf (robot description, URDF)
Before this commit: robot cubicbot_urdf, 10 links, 9 joints
Joints:
- joint left_wheel_joint: limit effort=100 velocity=100 -> (none); type continuous -> fixed
- joint lidar_joint: origin xyz=0 0 0.5 rpy=0 0 0 -> xyz=0 0 -0.32 rpy=0 0 0
- joint right_wheel_joint: limit effort=100 velocity=100 -> (none); type continuous -> fixed

File: demobot2_description/urdf/cubicbot/cubicbot_urdf_fixed.xacro (robot description, xacro)
@@ -1,5 +1,5 @@
 <?xml version="1.0"?>
-<robot name="circularbot_urdf" xmlns:xacro="http://www.ros.org/wiki/xacro">
-  <xacro:include filename="$(find demobot2_description)/urdf/circularbot/circularbot_essential.xacro" />
+<robot name="cubicbot_urdf" xmlns:xacro="http://www.ros.org/wiki/xacro">
+  <xacro:include filename="$(find demobot2_description)/urdf/cubicbot/cubicbot_essential.xacro" />
   <link name="base_footprint"/>
   <!-- base_link --> <!--Actual body/chassis of the robot-->
@@ -8,10 +8,10 @@
       <mass value="${base_mass}" />
       <origin xyz="0 0 0" />
-      <xacro:cylinder_inertia m="${base_mass}" r="${base_radius}" h="${base_height}" />
+      <xacro:box_inertia m="${base_mass}" x="${base_length}" y="${base_width}" z="${base_height}" />
     </inertial>
     <visual>
       <origin xyz="0 0 0" rpy="0 0 0" />
       <geometry>
-          <cylinder length="${base_height}" radius="${base_radius}" />
+          <box size="${base_length} ${base_width} ${base_height}" />
       </geometry>
       <material name="transyellow">
@@ -22,5 +22,5 @@
       <origin xyz="0 0 0" rpy="0 0 0 " />
       <geometry>
-          <cylinder length="${base_height}" radius="${base_radius}" />
+          <box size="${base_length} ${base_width} ${base_height}" />
       </geometry>
     </collision>
@@ -109,6 +109,6 @@
   </joint>
   <!-- Wheels -->
-  <xacro:wheel lr="left" parent="base_link" dir="1" z_offset="-0.43" roll="${-1.0 * M_PI_2}"/>
-  <xacro:wheel lr="right" parent="base_link" dir="-1" z_offset="-0.43" roll="${-1.0 * M_PI_2}"/>
+  <xacro:fixed_wheel lr="left" parent="base_link" dir="1" z_offset="-0.43" roll="${-1.0 * M_PI_2}"/>
+  <xacro:fixed_wheel lr="right" parent="base_link" dir="-1" z_offset="-0.43" roll="${-1.0 * M_PI_2}"/>
   <!-- Casters -->
   <xacro:caster fb="front" parent="base_link" dir="1" z_offset="-0.449" roll="0" color="Red"/>

File: demobot2_description/urdf/demobot/demobot_essential.xacro (robot description, xacro)
@@ -61,6 +61,6 @@
         <origin xyz="0 0 0" rpy="0 0 0 " />
         <geometry>
-          <!-- <cylinder length="${wheel_height}" radius="${wheel_radius}" /> -->
-          <mesh filename="package://demobot2_description/meshes/demobot/wheel.stl"/>
+          <cylinder length="${wheel_height}" radius="${wheel_radius}" />
+          <!-- <mesh filename="package://demobot2_description/meshes/demobot/wheel.stl"/> -->
         </geometry>
         <material name="Black" />
@@ -87,3 +87,32 @@
     </joint>
   </xacro:macro>
+  <!-- Visualization for real robot -->
+  <xacro:macro name="fixed_wheel" params="lr parent dir z_offset roll"> <!-- lr: left, right -->
+    <link name="${lr}_wheel_link">
+      <visual>
+        <origin xyz="0 0 0" rpy="0 0 0 " />
+        <geometry>
+          <cylinder length="${wheel_height}" radius="${wheel_radius}" />
+        </geometry>
+        <material name="Black" />
+      </visual>
+      <collision>
+        <origin xyz="0 0 0" rpy="0 0 0 " />
+        <geometry>
+          <cylinder length="${wheel_height}" radius="${wheel_radius}" />
+        </geometry>
+      </collision>
+      <inertial>
+        <mass value="${wheel_mass}" />
+        <origin xyz="0 0 0" />
+        <xacro:cylinder_inertia  m="${wheel_mass}" r="${wheel_radius}" h="${wheel_height}" />
+      </inertial>
+    </link>
+    <joint name="${lr}_wheel_joint" type="fixed">
+      <parent link="${parent}"/>
+      <child link="${lr}_wheel_link"/>
+      <origin xyz="0 ${dir * wheel_spacing / 2} ${z_offset}" rpy="${roll} 0 0" />
+      <axis xyz="0 0 1" rpy="0 0 0" />
+    </joint>
+  </xacro:macro>
 </robot>

File: demobot2_description/urdf/demobot/demobot_gazebo.urdf (robot description, URDF)
Before this commit: robot demobot_gazebo, 7 links, 6 joints
Links:
- link base_link: geometry collision box size=0.24 0.2 0.02; visual box size=0.24 0.2 0.02
- link left_wheel_link: geometry collision cylinder length=0.035 radius=0.0365; visual cylinder length=0.035 radius=0.0365
- link right_wheel_link: geometry collision cylinder length=0.035 radius=0.0365; visual cylinder length=0.035 radius=0.0365
Joints:
- joint base_joint: origin xyz=0 0 00.0565 rpy=0 0 0 -> xyz=0 0 0.0565 rpy=0 0 0
- joint lidar_joint: origin xyz=0 0 0.3 rpy=0 0 0 -> xyz=0 0 0.105 rpy=0 0 0

File: demobot2_description/urdf/demobot/demobot_gazebo.xacro (robot description, xacro)
@@ -5,5 +5,8 @@
   <xacro:arg name="lidar_visual"    default="false"/>
   <gazebo reference="base_link">
-    <material>Gazebo/White</material>
+    <material>Gazebo/Yellow</material>
+    <visual>
+      <transparency>0.3</transparency>
+    </visual>
   </gazebo>
   <gazebo reference="left_wheel_link">
@@ -108,5 +111,5 @@
       <publish_odom>true</publish_odom>
       <publish_odom_tf>true</publish_odom_tf>
-      <publish_wheel_tf>false</publish_wheel_tf>
+      <publish_wheel_tf>true</publish_wheel_tf>
       <odometry_topic>odom</odometry_topic>
       <odometry_frame>odom</odometry_frame>

File: demobot2_description/urdf/demobot/demobot_urdf.xacro (robot description, xacro)
@@ -11,13 +11,15 @@
     </inertial>     -->
     <visual>
-      <origin xyz="0 0 0" rpy="0 0 0" />
+      <origin xyz="-0.06 0 0.05" rpy="0 0 0" />
       <geometry>
-          <!-- <box size="${base_length} ${base_width} ${base_height}" /> -->
-          <mesh filename="package://demobot2_description/meshes/demobot/body.stl"/>
+          <box size="${base_length} ${base_width} ${base_height}" />
+          <!-- <mesh filename="package://demobot2_description/meshes/demobot/body.stl"/> -->
       </geometry>
-      <material name="White" />
+      <material name="transyellow">
+        <color rgba="1.0 1.0 0.0 0.3"/>
+      </material>
     </visual>
     <collision>
-      <origin xyz="0 0 0" rpy="0 0 0 " />
+      <origin xyz="-0.06 0 0.05" rpy="0 0 0" />
       <geometry>
           <box size="${base_length} ${base_width} ${base_height}" />
@@ -69,5 +71,5 @@
       <parent link="base_footprint"/>
       <child link="base_link" />
-      <origin xyz="0 0 00.0565" rpy="0 0 0"/>
+      <origin xyz="0 0 0.0565" rpy="0 0 0"/>
   </joint>
   <joint name="caster_joint" type="fixed">
@@ -84,6 +86,5 @@
     <parent link="base_link"/>
     <child link="lidar_link"/>
-    <!-- <origin xyz="0 0 0.105" rpy="0 0 0"/> -->
-    <origin xyz="0 0 0.3" rpy="0 0 0"/>
+    <origin xyz="0 0 0.105" rpy="0 0 0"/> <!-- default z: 0.105 -->
   </joint>
   <!-- Wheels -->

File: demobot2_description/urdf/demobot/demobot_urdf_fixed.urdf (robot description, URDF)
Before this commit: robot demobot_urdf, 7 links, 6 joints
Links:
- link base_link: geometry collision box size=0.24 0.2 0.02; visual box size=0.24 0.2 0.02
- link left_wheel_link: geometry collision cylinder length=0.035 radius=0.0365; visual cylinder length=0.035 radius=0.0365
- link right_wheel_link: geometry collision cylinder length=0.035 radius=0.0365; visual cylinder length=0.035 radius=0.0365
Joints:
- joint base_joint: origin xyz=0 0 00.0565 rpy=0 0 0 -> xyz=0 0 0.0565 rpy=0 0 0
- joint left_wheel_joint: limit effort=100 velocity=100 -> (none); type continuous -> fixed
- joint lidar_joint: origin xyz=0 0 0.3 rpy=0 0 0 -> xyz=0 0 0.105 rpy=0 0 0
- joint right_wheel_joint: limit effort=100 velocity=100 -> (none); type continuous -> fixed

File: demobot2_description/urdf/demobot/demobot_urdf_fixed.xacro (robot description, xacro)
@@ -1,17 +1,18 @@
 <?xml version="1.0"?>
-<robot name="circularbot_urdf" xmlns:xacro="http://www.ros.org/wiki/xacro">
-  <xacro:include filename="$(find demobot2_description)/urdf/circularbot/circularbot_essential.xacro" />
+<robot name="demobot_urdf" xmlns:xacro="http://www.ros.org/wiki/xacro">
+  <xacro:include filename="$(find demobot2_description)/urdf/demobot/demobot_essential.xacro" />
   <link name="base_footprint"/>
   <!-- base_link --> <!--Actual body/chassis of the robot-->
   <link name="base_link">
-    <inertial>
+    <!-- <inertial>
       <mass value="${base_mass}" />
       <origin xyz="0 0 0" />
-      <xacro:cylinder_inertia m="${base_mass}" r="${base_radius}" h="${base_height}" />
-    </inertial>
+        <box_inertia  />
+    </inertial>     -->
     <visual>
-      <origin xyz="0 0 0" rpy="0 0 0" />
+      <origin xyz="-0.06 0 0.05" rpy="0 0 0" />
       <geometry>
-          <cylinder length="${base_height}" radius="${base_radius}" />
+          <box size="${base_length} ${base_width} ${base_height}" />
+          <!-- <mesh filename="package://demobot2_description/meshes/demobot/body.stl"/> -->
       </geometry>
       <material name="transyellow">
@@ -20,12 +21,12 @@
     </visual>
     <collision>
-      <origin xyz="0 0 0" rpy="0 0 0 " />
+      <origin xyz="-0.06 0 0.05" rpy="0 0 0" />
       <geometry>
-          <cylinder length="${base_height}" radius="${base_radius}" />
+          <box size="${base_length} ${base_width} ${base_height}" />
       </geometry>
     </collision>
   </link>
   <!-- caster -->
-  <!-- <link name="caster_link">
+  <link name="caster_link">
     <visual>
       <origin xyz="0 0 0" rpy="0 0 0" />
@@ -48,7 +49,7 @@
                izz="0.001" />
     </inertial>
-  </link> -->
+  </link>
   <link name="imu_link">
-    <visual>
+      <visual>
       <origin xyz="0 0 0" rpy="0 0 0" />
       <geometry>
@@ -59,5 +60,5 @@
   </link>
   <link name="lidar_link">
-    <visual>
+      <visual>
       <origin xyz="0 0 0" rpy="0 0 0" />
       <geometry>
@@ -67,50 +68,26 @@
     </visual>
   </link>
-  <link name="camera_link">
-    <visual>
-      <origin xyz="0 0 0" rpy="0 0 0" />
-      <geometry>
-	      <box size="${camera_length} ${camera_width} ${camera_height}" />
-      </geometry>
-      <material name="Red" />
-    </visual>
-  </link>
-  <link name="depth_camera_link">
-  </link>
   <joint name="base_joint" type="fixed">
       <parent link="base_footprint"/>
       <child link="base_link" />
-      <origin xyz="0 0 0.5" rpy="0 0 0"/>
+      <origin xyz="0 0 0.0565" rpy="0 0 0"/>
   </joint>
-  <!-- <joint name="caster_joint" type="fixed">
+  <joint name="caster_joint" type="fixed">
     <parent link="base_link"/>
     <child link="caster_link"/>
     <origin xyz="-0.15 0.0 -0.0465" rpy="0 0 0"/>
-  </joint> -->
+  </joint>
   <joint name="imu_joint" type="fixed">
     <parent link="base_link"/>
     <child link="imu_link"/>
-    <origin xyz="0.0 0.0 -0.4" rpy="0 0 0"/>
+    <origin xyz="0.0 0.0 0.075" rpy="0 0 0"/>
   </joint>
   <joint name="lidar_joint" type="fixed">
     <parent link="base_link"/>
     <child link="lidar_link"/>
-    <origin xyz="0 0 -0.32" rpy="0 0 0"/> <!-- default z: -0.32 -->
-  </joint>
-  <joint name="camera_joint" type="fixed">
-    <parent link="base_link"/>
-    <child link="camera_link"/>
-    <origin xyz="0.31 0 0" rpy="0 0 0"/>
-  </joint>
-  <joint name="depth_camera_joint" type="fixed">
-    <parent link="base_link"/>
-    <child link="depth_camera_link"/>
-    <origin xyz="0.31 0 0" rpy="${-1.0 * M_PI_2} 0 ${-1.0 * M_PI_2}"/>
+    <origin xyz="0 0 0.105" rpy="0 0 0"/> <!-- default z: 0.105 -->
   </joint>
   <!-- Wheels -->
-  <xacro:wheel lr="left" parent="base_link" dir="1" z_offset="-0.43" roll="${-1.0 * M_PI_2}"/>
-  <xacro:wheel lr="right" parent="base_link" dir="-1" z_offset="-0.43" roll="${-1.0 * M_PI_2}"/>
-  <!-- Casters -->
-  <xacro:caster fb="front" parent="base_link" dir="1" z_offset="-0.449" roll="0" color="Red"/>
-  <xacro:caster fb="back" parent="base_link" dir="-1" z_offset="-0.449" roll="0" color="Blue"/>
+  <xacro:fixed_wheel lr="left" parent="base_link" dir="1" z_offset="-0.02" roll="${-1.0 * M_PI_2}"/>
+  <xacro:fixed_wheel lr="right" parent="base_link" dir="-1" z_offset="-0.02" roll="${-1.0 * M_PI_2}"/>
 </robot>
