Commit message: modify tf w.r.t REP105 & add robot locolization

File: demobot2_description/urdf/circularbot/circularbot_gazebo.xacro (robot description, xacro)
@@ -127,5 +127,5 @@
       <odometry_topic>odom</odometry_topic>
       <odometry_frame>odom</odometry_frame>
-      <robot_base_frame>base_footprint</robot_base_frame>
+      <robot_base_frame>base_link</robot_base_frame>
     </plugin>
   </gazebo>

File: demobot2_description/urdf/circularbot/circularbot_urdf.xacro (robot description, xacro)
@@ -79,7 +79,7 @@
   </link>
   <joint name="base_joint" type="fixed">
-      <parent link="base_footprint"/>
-      <child link="base_link" />
-      <origin xyz="0 0 0.5" rpy="0 0 0"/>
+      <parent link="base_link"/>
+      <child link="base_footprint" />
+      <origin xyz="0 0 -0.5" rpy="0 0 0"/>
   </joint>
   <!-- <joint name="caster_joint" type="fixed">

File: demobot2_description/urdf/circularbot/circularbot_urdf_fixed.xacro (robot description, xacro)
@@ -79,7 +79,7 @@
   </link>
   <joint name="base_joint" type="fixed">
-      <parent link="base_footprint"/>
-      <child link="base_link" />
-      <origin xyz="0 0 0.5" rpy="0 0 0"/>
+      <parent link="base_link"/>
+      <child link="base_footprint" />
+      <origin xyz="0 0 -0.5" rpy="0 0 0"/>
   </joint>
   <!-- <joint name="caster_joint" type="fixed">

File: demobot2_description/urdf/cubicbot/cubicbot_gazebo.xacro (robot description, xacro)
@@ -127,5 +127,5 @@
       <odometry_topic>odom</odometry_topic>
       <odometry_frame>odom</odometry_frame>
-      <robot_base_frame>base_footprint</robot_base_frame>
+      <robot_base_frame>base_link</robot_base_frame>
     </plugin>
   </gazebo>

File: demobot2_description/urdf/cubicbot/cubicbot_urdf.xacro (robot description, xacro)
@@ -79,7 +79,7 @@
   </link>
   <joint name="base_joint" type="fixed">
-      <parent link="base_footprint"/>
-      <child link="base_link" />
-      <origin xyz="0 0 0.5" rpy="0 0 0"/>
+      <parent link="base_link"/>
+      <child link="base_footprint" />
+      <origin xyz="0 0 -0.5" rpy="0 0 0"/>
   </joint>
   <!-- <joint name="caster_joint" type="fixed">

File: demobot2_description/urdf/cubicbot/cubicbot_urdf_fixed.xacro (robot description, xacro)
@@ -79,7 +79,7 @@
   </link>
   <joint name="base_joint" type="fixed">
-      <parent link="base_footprint"/>
-      <child link="base_link" />
-      <origin xyz="0 0 0.5" rpy="0 0 0"/>
+      <parent link="base_link"/>
+      <child link="base_footprint" />
+      <origin xyz="0 0 -0.5" rpy="0 0 0"/>
   </joint>
   <!-- <joint name="caster_joint" type="fixed">

File: demobot2_description/urdf/demobot/demobot_gazebo.xacro (robot description, xacro)
@@ -114,5 +114,5 @@
       <odometry_topic>odom</odometry_topic>
       <odometry_frame>odom</odometry_frame>
-      <robot_base_frame>base_footprint</robot_base_frame>
+      <robot_base_frame>base_link</robot_base_frame>
     </plugin>
   </gazebo>

File: demobot2_description/urdf/demobot/demobot_urdf.xacro (robot description, xacro)
@@ -69,7 +69,7 @@
   </link>
   <joint name="base_joint" type="fixed">
-      <parent link="base_footprint"/>
-      <child link="base_link" />
-      <origin xyz="0 0 0.0565" rpy="0 0 0"/>
+      <parent link="base_link"/>
+      <child link="base_footprint" />
+      <origin xyz="0 0 -0.0565" rpy="0 0 0"/>
   </joint>
   <joint name="caster_joint" type="fixed">

File: demobot2_description/urdf/demobot/demobot_urdf_fixed.xacro (robot description, xacro)
@@ -69,7 +69,7 @@
   </link>
   <joint name="base_joint" type="fixed">
-      <parent link="base_footprint"/>
-      <child link="base_link" />
-      <origin xyz="0 0 0.0565" rpy="0 0 0"/>
+      <parent link="base_link"/>
+      <child link="base_footprint" />
+      <origin xyz="0 0 -0.0565" rpy="0 0 0"/>
   </joint>
   <joint name="caster_joint" type="fixed">

Commit message: udpate urdf

File: demobot2_description/urdf/circularbot/circularbot_gazebo.xacro (robot description, xacro)
@@ -5,7 +5,4 @@
   <xacro:arg name="lidar_visual"    default="false"/>
   <!-- gazebo reference="xxx_link" 是指给xxx_link赋予属性(颜色,摩擦力等)或添加插件(传感器,控制等)-->
-  <gazebo reference="camera_link">
-    <material>Gazebo/Red</material>
-  </gazebo>
   <gazebo reference="base_link">
     <material>Gazebo/Yellow</material>
@@ -60,7 +57,5 @@
       <plugin name="imu_plugin" filename="libgazebo_ros_imu_sensor.so">
         <ros>
-          <!-- publish to /imu/data -->
-          <!-- <namespace>/imu</namespace>
-          <remapping>~/out:=data</remapping> -->
+          <!-- <namespace>/sensors</namespace> -->
           <remapping>~/out:=imu_data</remapping>
         </ros>
@@ -95,12 +90,48 @@
         </noise>
       </ray>
-      <plugin name="lidar_plugin" filename="libgazebo_ros_ray_sensor.so">
+      <plugin name="scan" filename="libgazebo_ros_ray_sensor.so">
         <ros>
-            <!-- <namespace>/scan</namespace>
-            <remapping>~/out:=data</remapping> -->
+            <!-- <namespace>/sensors</namespace> -->
             <remapping>~/out:=scan</remapping>
         </ros>
         <output_type>sensor_msgs/LaserScan</output_type>
         <frame_name>lidar_link</frame_name>
+      </plugin>
+    </sensor>
+  </gazebo>
+  <gazebo reference="camera_link">
+    <material>Gazebo/Red</material>
+    <sensor name="depth_camera" type="depth">
+      <visualize>true</visualize>
+      <update_rate>30.0</update_rate>
+      <camera name="camera">
+        <horizontal_fov>1.047198</horizontal_fov>
+        <image>
+          <width>640</width>
+          <height>480</height>
+          <format>R8G8B8</format>
+        </image>
+        <clip>
+          <near>0.05</near>
+          <far>3</far>
+        </clip>
+      </camera>
+      <plugin name="depth_camera_controller" filename="libgazebo_ros_camera.so">
+        <baseline>0.2</baseline>
+        <alwaysOn>true</alwaysOn>
+        <updateRate>0.0</updateRate>
+        <frame_name>camera_depth_frame</frame_name>
+        <pointCloudCutoff>0.5</pointCloudCutoff>
+        <pointCloudCutoffMax>3.0</pointCloudCutoffMax>
+        <distortionK1>0</distortionK1>
+        <distortionK2>0</distortionK2>
+        <distortionK3>0</distortionK3>
+        <distortionT1>0</distortionT1>
+        <distortionT2>0</distortionT2>
+        <CxPrime>0</CxPrime>
+        <Cx>0</Cx>
+        <Cy>0</Cy>
+        <focalLength>0</focalLength>
+        <hackBaseline>0</hackBaseline>
       </plugin>
     </sensor>

File: demobot2_description/urdf/circularbot/circularbot_urdf.xacro (robot description, xacro)
@@ -26,27 +26,4 @@
     </collision>
   </link>
-  <!-- caster -->
-  <!-- <link name="caster_link">
-    <visual>
-      <origin xyz="0 0 0" rpy="0 0 0" />
-      <geometry>
-	      <sphere radius="${caster_radius}" />
-      </geometry>
-      <material name="Black" />
-    </visual>
-    <collision>
-      <origin xyz="0 0 0" rpy="0 0 0" />
-      <geometry>
-	        <sphere radius="${caster_radius}" />
-      </geometry>
-    </collision>
-    <inertial>
-      <mass value="${caster_mass}" />
-      <origin xyz="0 0 0" />
-      <inertia ixx="0.001" ixy="0.0" ixz="0.0"
-               iyy="0.001" iyz="0.0"
-               izz="0.001" />
-    </inertial>
-  </link> -->
   <link name="imu_link">
     <visual>
@@ -75,7 +52,17 @@
       <material name="Red" />
     </visual>
+    <collision>
+      <origin xyz="0 0 0" rpy="0 0 0 " />
+      <geometry>
+        <box size="${camera_length} ${camera_width} ${camera_height}" />
+      </geometry>
+    </collision>
+    <inertial>
+      <mass value="${camera_mass}" />
+      <origin xyz="0 0 0" />
+      <xacro:box_inertia m="${camera_mass}" x="${camera_length}" y="${camera_width}" z="${camera_height}" />
+    </inertial>
   </link>
-  <link name="depth_camera_link">
-  </link>
+  <link name="camera_depth_frame"/>
   <joint name="base_joint" type="fixed">
       <parent link="base_link"/>
@@ -83,9 +70,4 @@
       <origin xyz="0 0 -0.5" rpy="0 0 0"/>
   </joint>
-  <!-- <joint name="caster_joint" type="fixed">
-    <parent link="base_link"/>
-    <child link="caster_link"/>
-    <origin xyz="-0.15 0.0 -0.0465" rpy="0 0 0"/>
-  </joint> -->
   <joint name="imu_joint" type="fixed">
     <parent link="base_link"/>
@@ -103,8 +85,8 @@
     <origin xyz="0.31 0 0" rpy="0 0 0"/>
   </joint>
-  <joint name="depth_camera_joint" type="fixed">
-    <parent link="base_link"/>
-    <child link="depth_camera_link"/>
-    <origin xyz="0.31 0 0" rpy="${-1.0 * M_PI_2} 0 ${-1.0 * M_PI_2}"/>
+  <joint name="camera_depth_joint" type="fixed">
+    <parent link="camera_link"/>
+    <child link="camera_depth_frame"/>
+    <origin xyz="0.0 0 0" rpy="${-1.0 * M_PI_2} 0 ${-1.0 * M_PI_2}"/>
   </joint>
   <!-- Wheels -->

File: demobot2_description/urdf/circularbot/circularbot_urdf_fixed.xacro (robot description, xacro)
@@ -26,27 +26,4 @@
     </collision>
   </link>
-  <!-- caster -->
-  <!-- <link name="caster_link">
-    <visual>
-      <origin xyz="0 0 0" rpy="0 0 0" />
-      <geometry>
-	      <sphere radius="${caster_radius}" />
-      </geometry>
-      <material name="Black" />
-    </visual>
-    <collision>
-      <origin xyz="0 0 0" rpy="0 0 0" />
-      <geometry>
-	        <sphere radius="${caster_radius}" />
-      </geometry>
-    </collision>
-    <inertial>
-      <mass value="${caster_mass}" />
-      <origin xyz="0 0 0" />
-      <inertia ixx="0.001" ixy="0.0" ixz="0.0"
-               iyy="0.001" iyz="0.0"
-               izz="0.001" />
-    </inertial>
-  </link> -->
   <link name="imu_link">
     <visual>
@@ -76,6 +53,5 @@
     </visual>
   </link>
-  <link name="depth_camera_link">
-  </link>
+  <link name="camera_depth_frame"/>
   <joint name="base_joint" type="fixed">
       <parent link="base_link"/>
@@ -83,9 +59,4 @@
       <origin xyz="0 0 -0.5" rpy="0 0 0"/>
   </joint>
-  <!-- <joint name="caster_joint" type="fixed">
-    <parent link="base_link"/>
-    <child link="caster_link"/>
-    <origin xyz="-0.15 0.0 -0.0465" rpy="0 0 0"/>
-  </joint> -->
   <joint name="imu_joint" type="fixed">
     <parent link="base_link"/>
@@ -103,8 +74,8 @@
     <origin xyz="0.31 0 0" rpy="0 0 0"/>
   </joint>
-  <joint name="depth_camera_joint" type="fixed">
-    <parent link="base_link"/>
-    <child link="depth_camera_link"/>
-    <origin xyz="0.31 0 0" rpy="${-1.0 * M_PI_2} 0 ${-1.0 * M_PI_2}"/>
+  <joint name="camera_depth_joint" type="fixed">
+    <parent link="camera_link"/>
+    <child link="camera_depth_frame"/>
+    <origin xyz="0.0 0 0" rpy="${-1.0 * M_PI_2} 0 ${-1.0 * M_PI_2}"/>
   </joint>
   <!-- Wheels -->

File: demobot2_description/urdf/cubicbot/cubicbot_gazebo.xacro (robot description, xacro)
@@ -5,7 +5,4 @@
   <xacro:arg name="lidar_visual"    default="false"/>
   <!-- gazebo reference="xxx_link" 是指给xxx_link赋予属性(颜色,摩擦力等)或添加插件(传感器,控制等)-->
-  <gazebo reference="camera_link">
-    <material>Gazebo/Red</material>
-  </gazebo>
   <gazebo reference="base_link">
     <material>Gazebo/Yellow</material>
@@ -60,7 +57,5 @@
       <plugin name="imu_plugin" filename="libgazebo_ros_imu_sensor.so">
         <ros>
-          <!-- publish to /imu/data -->
-          <!-- <namespace>/imu</namespace>
-          <remapping>~/out:=data</remapping> -->
+          <!-- <namespace>/sensors</namespace> -->
           <remapping>~/out:=imu_data</remapping>
         </ros>
@@ -74,5 +69,5 @@
       <visualize>true</visualize>
       <pose>0 0 0 0 0 0</pose>
-      <update_rate>10</update_rate>
+      <update_rate>15</update_rate>
       <ray>
         <scan>
@@ -95,12 +90,48 @@
         </noise>
       </ray>
-      <plugin name="lidar_plugin" filename="libgazebo_ros_ray_sensor.so">
+      <plugin name="scan" filename="libgazebo_ros_ray_sensor.so">
         <ros>
-            <!-- <namespace>/scan</namespace>
-            <remapping>~/out:=data</remapping> -->
+            <!-- <namespace>/sensors</namespace> -->
             <remapping>~/out:=scan</remapping>
         </ros>
         <output_type>sensor_msgs/LaserScan</output_type>
         <frame_name>lidar_link</frame_name>
+      </plugin>
+    </sensor>
+  </gazebo>
+  <gazebo reference="camera_link">
+    <material>Gazebo/Red</material>
+    <sensor name="depth_camera" type="depth">
+      <visualize>true</visualize>
+      <update_rate>15.0</update_rate>
+      <camera name="camera">
+        <horizontal_fov>1.047198</horizontal_fov>
+        <image>
+          <width>160</width>
+          <height>120</height>
+          <format>R8G8B8</format>
+        </image>
+        <clip>
+          <near>0.05</near>
+          <far>3</far>
+        </clip>
+      </camera>
+      <plugin name="depth_camera_controller" filename="libgazebo_ros_camera.so">
+        <baseline>0.2</baseline>
+        <alwaysOn>true</alwaysOn>
+        <updateRate>0.0</updateRate>
+        <frame_name>depth_camera_link</frame_name>
+        <pointCloudCutoff>0.5</pointCloudCutoff>
+        <pointCloudCutoffMax>3.0</pointCloudCutoffMax>
+        <distortionK1>0</distortionK1>
+        <distortionK2>0</distortionK2>
+        <distortionK3>0</distortionK3>
+        <distortionT1>0</distortionT1>
+        <distortionT2>0</distortionT2>
+        <CxPrime>0</CxPrime>
+        <Cx>0</Cx>
+        <Cy>0</Cy>
+        <focalLength>0</focalLength>
+        <hackBaseline>0</hackBaseline>
       </plugin>
     </sensor>

File: demobot2_description/urdf/cubicbot/cubicbot_urdf.xacro (robot description, xacro)
@@ -26,27 +26,4 @@
     </collision>
   </link>
-  <!-- caster -->
-  <!-- <link name="caster_link">
-    <visual>
-      <origin xyz="0 0 0" rpy="0 0 0" />
-      <geometry>
-	      <sphere radius="${caster_radius}" />
-      </geometry>
-      <material name="Black" />
-    </visual>
-    <collision>
-      <origin xyz="0 0 0" rpy="0 0 0" />
-      <geometry>
-	        <sphere radius="${caster_radius}" />
-      </geometry>
-    </collision>
-    <inertial>
-      <mass value="${caster_mass}" />
-      <origin xyz="0 0 0" />
-      <inertia ixx="0.001" ixy="0.0" ixz="0.0"
-               iyy="0.001" iyz="0.0"
-               izz="0.001" />
-    </inertial>
-  </link> -->
   <link name="imu_link">
     <visual>
@@ -75,4 +52,15 @@
       <material name="Red" />
     </visual>
+    <collision>
+      <origin xyz="0 0 0" rpy="0 0 0 " />
+      <geometry>
+        <box size="${camera_length} ${camera_width} ${camera_height}" />
+      </geometry>
+    </collision>
+    <inertial>
+      <mass value="${camera_mass}" />
+      <origin xyz="0 0 0" />
+      <xacro:box_inertia m="${camera_mass}" x="${camera_length}" y="${camera_width}" z="${camera_height}" />
+    </inertial>
   </link>
   <link name="depth_camera_link">
@@ -83,9 +71,4 @@
       <origin xyz="0 0 -0.5" rpy="0 0 0"/>
   </joint>
-  <!-- <joint name="caster_joint" type="fixed">
-    <parent link="base_link"/>
-    <child link="caster_link"/>
-    <origin xyz="-0.15 0.0 -0.0465" rpy="0 0 0"/>
-  </joint> -->
   <joint name="imu_joint" type="fixed">
     <parent link="base_link"/>
@@ -104,7 +87,7 @@
   </joint>
   <joint name="depth_camera_joint" type="fixed">
-    <parent link="base_link"/>
+    <parent link="camera_link"/>
     <child link="depth_camera_link"/>
-    <origin xyz="0.31 0 0" rpy="${-1.0 * M_PI_2} 0 ${-1.0 * M_PI_2}"/>
+    <origin xyz="0 0 0" rpy="${-1.0 * M_PI_2} 0 ${-1.0 * M_PI_2}"/>
   </joint>
   <!-- Wheels -->

File: demobot2_description/urdf/cubicbot/cubicbot_urdf_fixed.xacro (robot description, xacro)
@@ -26,27 +26,4 @@
     </collision>
   </link>
-  <!-- caster -->
-  <!-- <link name="caster_link">
-    <visual>
-      <origin xyz="0 0 0" rpy="0 0 0" />
-      <geometry>
-	      <sphere radius="${caster_radius}" />
-      </geometry>
-      <material name="Black" />
-    </visual>
-    <collision>
-      <origin xyz="0 0 0" rpy="0 0 0" />
-      <geometry>
-	        <sphere radius="${caster_radius}" />
-      </geometry>
-    </collision>
-    <inertial>
-      <mass value="${caster_mass}" />
-      <origin xyz="0 0 0" />
-      <inertia ixx="0.001" ixy="0.0" ixz="0.0"
-               iyy="0.001" iyz="0.0"
-               izz="0.001" />
-    </inertial>
-  </link> -->
   <link name="imu_link">
     <visual>
@@ -83,9 +60,4 @@
       <origin xyz="0 0 -0.5" rpy="0 0 0"/>
   </joint>
-  <!-- <joint name="caster_joint" type="fixed">
-    <parent link="base_link"/>
-    <child link="caster_link"/>
-    <origin xyz="-0.15 0.0 -0.0465" rpy="0 0 0"/>
-  </joint> -->
   <joint name="imu_joint" type="fixed">
     <parent link="base_link"/>
@@ -104,7 +76,7 @@
   </joint>
   <joint name="depth_camera_joint" type="fixed">
-    <parent link="base_link"/>
+    <parent link="camera_link"/>
     <child link="depth_camera_link"/>
-    <origin xyz="0.31 0 0" rpy="${-1.0 * M_PI_2} 0 ${-1.0 * M_PI_2}"/>
+    <origin xyz="0 0 0" rpy="${-1.0 * M_PI_2} 0 ${-1.0 * M_PI_2}"/>
   </joint>
   <!-- Wheels -->

File: demobot2_description/urdf/demobot/demobot_gazebo.xacro (robot description, xacro)
@@ -47,7 +47,5 @@
       <plugin name="imu_plugin" filename="libgazebo_ros_imu_sensor.so">
         <ros>
-          <!-- publish to /imu/data -->
-          <!-- <namespace>/imu</namespace>
-          <remapping>~/out:=data</remapping> -->
+          <!-- <namespace>/sensors</namespace> -->
           <remapping>~/out:=imu_data</remapping>
         </ros>
@@ -84,6 +82,5 @@
       <plugin name="lidar_plugin" filename="libgazebo_ros_ray_sensor.so">
         <ros>
-            <!-- <namespace>/scan</namespace>
-            <remapping>~/out:=data</remapping> -->
+            <!-- <namespace>/sensors</namespace> -->
             <remapping>~/out:=scan</remapping>
         </ros>
