Commit message: try keepout zone

File: demobot2_description/urdf/circularbot/circularbot_urdf.xacro (robot description, xacro)
@@ -5,9 +5,10 @@
   <!-- base_link --> <!--Actual body/chassis of the robot-->
   <link name="base_link">
-    <inertial>
+    <!--KDL does not support a root link with an inertia.  As a workaround, you can add an extra dummy link to your URDF.-->
+    <!-- <inertial>
       <mass value="${base_mass}" />
       <origin xyz="0 0 0" />
       <xacro:cylinder_inertia m="${base_mass}" r="${base_radius}" h="${base_height}" />
-    </inertial>
+    </inertial> -->
     <visual>
       <origin xyz="0 0 0" rpy="0 0 0" />

File: demobot2_description/urdf/circularbot/circularbot_urdf_fixed.xacro (robot description, xacro)
@@ -5,9 +5,9 @@
   <!-- base_link --> <!--Actual body/chassis of the robot-->
   <link name="base_link">
-    <inertial>
+    <!-- <inertial>
       <mass value="${base_mass}" />
       <origin xyz="0 0 0" />
       <xacro:cylinder_inertia m="${base_mass}" r="${base_radius}" h="${base_height}" />
-    </inertial>
+    </inertial> -->
     <visual>
       <origin xyz="0 0 0" rpy="0 0 0" />
