Commit message: try different planner and controller

File: demobot2_description/urdf/cubicbot/cubicbot_essential.xacro (robot description, xacro)
@@ -25,5 +25,5 @@
   <xacro:property name="base_length" value="0.6" /> <!--m-->
   <xacro:property name="base_width" value="0.5" />
-  <xacro:property name="base_height" value="0.5" />
+  <xacro:property name="base_height" value="0.4" />
   <xacro:property name="base_mass" value="50" /> <!--kg-->
   <!-- Wheels -->

File: demobot2_description/urdf/cubicbot/cubicbot_gazebo.xacro (robot description, xacro)
@@ -67,5 +67,5 @@
     <sensor name="lidar_sensor" type="ray">
       <always_on>true</always_on>
-      <visualize>true</visualize>
+      <visualize>false</visualize>
       <pose>0 0 0 0 0 0</pose>
       <update_rate>15</update_rate>

File: demobot2_description/urdf/cubicbot/cubicbot_urdf.xacro (robot description, xacro)
@@ -5,9 +5,9 @@
   <!-- base_link --> <!--Actual body/chassis of the robot-->
   <link name="base_link">
-    <inertial>
+    <!-- <inertial>
       <mass value="${base_mass}" />
       <origin xyz="0 0 0" />
       <xacro:box_inertia m="${base_mass}" x="${base_length}" y="${base_width}" z="${base_height}" />
-    </inertial>
+    </inertial> -->
     <visual>
       <origin xyz="0 0 0" rpy="0 0 0" />

File: demobot2_description/urdf/cubicbot/cubicbot_urdf_fixed.xacro (robot description, xacro)
@@ -5,9 +5,9 @@
   <!-- base_link --> <!--Actual body/chassis of the robot-->
   <link name="base_link">
-    <inertial>
+    <!-- <inertial>
       <mass value="${base_mass}" />
       <origin xyz="0 0 0" />
       <xacro:box_inertia m="${base_mass}" x="${base_length}" y="${base_width}" z="${base_height}" />
-    </inertial>
+    </inertial> -->
     <visual>
       <origin xyz="0 0 0" rpy="0 0 0" />
